Commit message: Circumvent problem where joint oscillates by narrowing down joint range. Lower limit is 11 degrees off

File: kuka_kr6_r900sixx/urdf/kr6r900sixx_macro.xacro (robot description, xacro)
@@ -144,5 +144,6 @@
       <child link="${prefix}link_4"/>
       <axis xyz="-1 0 0"/>
-      <limit effort="100" lower="${-DEG2RAD * 185}" upper="${DEG2RAD * 185}" velocity="${DEG2RAD * 381}"/>
+      <limit effort="100" lower="${-DEG2RAD * 174}" upper="${DEG2RAD * 185}" velocity="${DEG2RAD * 381}"/>
+      <!--<limit effort="100" lower="${-DEG2RAD * 185}" upper="${DEG2RAD * 185}" velocity="${DEG2RAD * 381}"/>-->
     </joint>
     <joint name="${prefix}joint_a5" type="revolute">
